Commit message: [update] Adjust object URDF, MTL, and OBJ files to align with final experiment setup

File: assets/urdf/objects/cube_multicolor.urdf (robot description, URDF)
Before this commit: robot object, 1 links, 0 joints
Links:
- link object: geometry collision box size=0.04 0.04 0.04; visual mesh filename=meshes/cube_multicolor.obj scale=.5 .5 .5

File: assets/urdf/ycb/010_potted_meat_can/010_potted_meat_can.urdf (robot description, URDF)
Before this commit: robot potted_meat_can, 1 links, 0 joints
Links:
- link potted_meat_can: mass 0.026 -> 0.220; geometry collision mesh filename=ycb/010_potted_meat_can/collision.obj scale=0.006 0.006 0.006; visual mesh filename=ycb/010_potted_meat_can/textured.obj scale=0.006 0.006 0.006

File: assets/urdf/ycb/011_banana/011_banana.urdf (robot description, URDF)
Before this commit: robot banana, 1 links, 0 joints
Links:
- link banana: geometry collision mesh filename=ycb/011_banana/collision.obj scale=0.006 0.006 0.006; visual mesh filename=ycb/011_banana/textured.obj scale=0.006 0.006 0.006

File: assets/urdf/ycb/025_mug/025_mug.urdf (robot description, URDF)
Before this commit: robot mug, 1 links, 0 joints
Links:
- link mug: mass 0.102 -> 0.080; geometry collision mesh filename=ycb/025_mug/mug_collision.obj scale=0.006 0.006 0.006; visual mesh filename=ycb/025_mug/textured.obj scale=0.006 0.006 0.006

File: assets/urdf/ycb/061_foam_brick/061_foam_brick.urdf (robot description, URDF)
Before this commit: robot foam_brick, 1 links, 0 joints
Links:
- link foam_brick: geometry collision box scale=0.9 0.9 0.9 size=0.049 0.074 0.049; visual mesh filename=ycb/061_foam_brick/textured.obj scale=0.009 0.009 0.009
